Commit message: Uploading documentation

File: cat_model/urdf/cat.urdf (robot description, URDF)
Before this commit: robot cat, 9 links, 8 joints
Links:
- added link body, mass 1.1876; collision mesh filename=body.STL; visual mesh filename=body.STL
- link base_link: mass 1.1099 -> 0.00043835; geometry collision mesh filename=base_link.STL; visual mesh filename=base_link.STL
- link lowerleg_bl: mass 0.0699581201747257 -> 0.074855; geometry collision mesh filename=lowerleg_bl.STL; visual mesh filename=lowerleg_bl.STL
- link lowerleg_br: mass 0.0699581201944018 -> 0.074855; geometry collision mesh filename=lowerleg_br.STL; visual mesh filename=lowerleg_br.STL
- link lowerleg_fl: mass 0.0699581201554127 -> 0.074855; geometry collision mesh filename=lowerleg_fl.STL; visual mesh filename=lowerleg_fl.STL
- link lowerleg_fr: mass 0.0699581202170087 -> 0.074855; geometry collision mesh filename=lowerleg_fr.STL; visual mesh filename=lowerleg_fr.STL
- link upperleg_bl: mass 0.057335271066792 -> 0.061349; geometry collision mesh filename=upperleg_bl.STL; visual mesh filename=upperleg_bl.STL
- link upperleg_br: mass 0.0573352716458123 -> 0.061349; geometry collision mesh filename=upperleg_br.STL; visual mesh filename=upperleg_br.STL
- link upperleg_fl: mass 0.060463 -> 0.064696; geometry collision mesh filename=upperleg_fl.STL; visual mesh filename=upperleg_fl.STL
- link upperleg_fr: mass 0.060463 -> 0.064696; geometry collision mesh filename=upperleg_fr.STL; visual mesh filename=upperleg_fr.STL
Joints:
- added joint base_joint: type fixed, parent base_link, child body, origin xyz=-0.04859 0.11829 0.013453 rpy=1.5708 0 0, axis 0 0 0
- joint hip_bl: origin xyz=0.55677 -1.3166 0.72616 rpy=3.1416 -0.26336 0 -> xyz=-0.036159 -0.048413 0.15254 rpy=1.5708 0 0.28437; parent base_link -> body
- joint hip_br: origin xyz=0.55677 -1.2016 0.72616 rpy=-3.1416 -0.27684 0 -> xyz=-0.036159 -0.048413 0.037536 rpy=-1.5708 0 2.8638; parent base_link -> body
- joint hip_fl: origin xyz=0.72627 -1.3017 0.72616 rpy=-3.1416 0.77498 -3.1416 -> xyz=0.13334 -0.048413 0.13763 rpy=-1.5708 0 -2.3382; parent base_link -> body
- joint hip_fr: origin xyz=0.72627 -1.2165 0.72616 rpy=-3.1416 0.79756 -3.1416 -> xyz=0.13334 -0.048413 0.052443 rpy=1.5708 0 -0.80381; parent base_link -> body
- joint knee_bl: origin xyz=-0.015108 0 0.052884 rpy=0 -0.27249 0 -> xyz=-0.015108 0 0.052884 rpy=0 0.30565 -3.1416
- joint knee_br: origin xyz=-0.015108 0 0.052884 rpy=0 -0.29892 0 -> xyz=-0.015108 0 0.052884 rpy=0 0.27827 -3.1416
- joint knee_fl: origin xyz=0.039486 0 0.038287 rpy=0 -0.77368 3.1416 -> xyz=0.039486 0 0.038287 rpy=0 0.81927 0
- joint knee_fr: origin xyz=0.039486 0 0.038287 rpy=0 -0.81155 3.1416 -> xyz=0.039486 0 0.038287 rpy=0 0.79665 0
